Commit message: Updated version

File: ros2_ws/install/yahboom_rosmaster_description/share/yahboom_rosmaster_description/urdf/control/gazebo_sim_ros2_control.urdf.xacro (robot description, xacro)
@@ -1 +1,15 @@
-/home/amr01/fyp/ros2_ws/src/yahboom_rosmaster/yahboom_rosmaster_description/urdf/control/gazebo_sim_ros2_control.urdf.xacro
+<?xml version="1.0" ?>
+<robot xmlns:xacro="http://wiki.ros.org/xacro">
+    <xacro:macro name="load_gazebo_sim_ros2_control_plugin" params="robot_name use_gazebo">
+        <xacro:if value="${use_gazebo}">
+            <gazebo>
+                <plugin filename="gz_ros2_control-system" name="gz_ros2_control::GazeboSimROS2ControlPlugin">
+                    <parameters>$(find yahboom_rosmaster_description)/config/${robot_name}/ros2_controllers.yaml</parameters>
+                    <ros>
+                        <remapping>/controller_manager/robot_description:=/robot_description</remapping>
+                    </ros>
+                </plugin>
+            </gazebo>
+        </xacro:if>
+    </xacro:macro>
+</robot>

File: ros2_ws/install/yahboom_rosmaster_description/share/yahboom_rosmaster_description/urdf/control/rosmaster_x3_ros2_control.urdf.xacro (robot description, xacro)
@@ -1 +1,44 @@
-/home/amr01/fyp/ros2_ws/src/yahboom_rosmaster/yahboom_rosmaster_description/urdf/control/rosmaster_x3_ros2_control.urdf.xacro
+<?xml version="1.0" ?>
+<robot xmlns:xacro="http://wiki.ros.org/xacro">
+    <xacro:macro name="yahboom_rosmaster_ros2_control" params="prefix use_gazebo">
+        <ros2_control name="RobotSystem" type="system">
+            <hardware>
+                <xacro:if value="${use_gazebo}">
+                    <plugin>gz_ros2_control/GazeboSimSystem</plugin>
+                </xacro:if>
+            </hardware>
+            <joint name="${prefix}front_left_wheel_joint">
+              <command_interface name="velocity">
+                  <param name="min">-50.0</param>
+                  <param name="max">50.0</param>
+              </command_interface>
+              <state_interface name="position"/>
+              <state_interface name="velocity"/>
+          </joint>
+          <joint name="${prefix}front_right_wheel_joint">
+              <command_interface name="velocity">
+                  <param name="min">-50.0</param>
+                  <param name="max">50.0</param>
+              </command_interface>
+              <state_interface name="position"/>
+              <state_interface name="velocity"/>
+          </joint>
+          <joint name="${prefix}back_left_wheel_joint">
+              <command_interface name="velocity">
+                  <param name="min">-50.0</param>
+                  <param name="max">50.0</param>
+              </command_interface>
+              <state_interface name="position"/>
+              <state_interface name="velocity"/>
+          </joint>
+          <joint name="${prefix}back_right_wheel_joint">
+              <command_interface name="velocity">
+                  <param name="min">-50.0</param>
+                  <param name="max">50.0</param>
+              </command_interface>
+              <state_interface name="position"/>
+              <state_interface name="velocity"/>
+          </joint>
+      </ros2_control>
+  </xacro:macro>
+</robot>

File: ros2_ws/install/yahboom_rosmaster_description/share/yahboom_rosmaster_description/urdf/control/velocity_control_plugin.urdf.xacro (robot description, xacro)
@@ -1 +1,16 @@
-/home/amr01/fyp/ros2_ws/src/yahboom_rosmaster/yahboom_rosmaster_description/urdf/control/velocity_control_plugin.urdf.xacro
+<?xml version="1.0"?>
+<robot xmlns:xacro="http://www.ros.org/wiki/xacro">
+    <xacro:macro name="load_velocity_control_plugin" params="use_gazebo">
+        <xacro:if value="${use_gazebo}">
+            <gazebo>
+                <plugin
+                    filename="gz-sim-velocity-control-system"
+                    name="gz::sim::systems::VelocityControl">
+                    <topic>mecanum_drive_controller/cmd_vel</topic>
+                    <initial_linear>0 0 0</initial_linear>
+                    <initial_angular>0 0 0</initial_angular>
+                </plugin>
+            </gazebo>
+        </xacro:if>
+    </xacro:macro>
+</robot>

File: ros2_ws/install/yahboom_rosmaster_description/share/yahboom_rosmaster_description/urdf/mech/mecanum_wheel.urdf.xacro (robot description, xacro)
@@ -1 +1,60 @@
-/home/amr01/fyp/ros2_ws/src/yahboom_rosmaster/yahboom_rosmaster_description/urdf/mech/mecanum_wheel.urdf.xacro
+<?xml version="1.0"?>
+<robot xmlns:xacro="http://www.ros.org/wiki/xacro">
+  <xacro:property name="wheel_radius" value="0.0325" />
+  <xacro:property name="wheel_separation" value="0.169" />
+  <xacro:property name="wheel_width" value="0.03040" />
+  <xacro:property name="wheel_mass" value="9.1" />
+  <xacro:property name="wheel_xoff" value="0.08" />
+  <xacro:property name="wheel_yoff" value="-0.01" />
+  <xacro:macro name="mecanum_wheel" params="prefix side x_reflect y_reflect">
+    <link name="${prefix}${side}_wheel_link">
+      <visual>
+        <origin xyz="0 0 0" rpy="${pi/2} 0 0"/>
+        <geometry>
+          <mesh filename="file://$(find yahboom_rosmaster_description)/meshes/rosmaster_x3/visual/${side}_wheel_X3.STL"/>
+        </geometry>
+        <material name="dark_gray">
+          <color rgba="0.2 0.2 0.2 1.0"/>
+        </material>
+      </visual>
+      <collision>
+        <origin xyz="0 0 0" rpy="${pi/2} 0 0"/>
+        <geometry>
+          <cylinder radius="${wheel_radius}" length="${wheel_width}"/>
+        </geometry>
+      </collision>
+      <inertial>
+        <origin xyz="0 0 0" rpy="0 0 0"/>
+        <mass value="${wheel_mass}"/>
+        <inertia
+          ixx="${(wheel_mass/12.0) * (3*wheel_radius*wheel_radius + wheel_width*wheel_width)}" ixy="0" ixz="0"
+          iyy="${(wheel_mass/2.0) * (wheel_radius*wheel_radius)}" iyz="0"
+          izz="${(wheel_mass/12.0) * (3*wheel_radius*wheel_radius + wheel_width*wheel_width)}"/>
+      </inertial>
+    </link>
+    <joint name="${prefix}${side}_wheel_joint" type="continuous">
+      <axis xyz="0 1 0"/>
+      <parent link="${prefix}base_link"/>
+      <child link="${prefix}${side}_wheel_link"/>
+      <origin xyz="${x_reflect*wheel_xoff} ${y_reflect*(wheel_separation/2+wheel_yoff)} ${-wheel_radius}" rpy="0 0 0"/>
+    </joint>
+    <gazebo reference="${prefix}${side}_wheel_link">
+      <surface>
+        <friction>
+          <ode>
+              <mu>1.0</mu>
+              <mu2>0.0</mu2>
+          </ode>
+        </friction>
+      </surface>
+      <visual>
+          <material>
+              <ambient>0.2 0.2 0.2 1.0</ambient>
+              <diffuse>0.2 0.2 0.2 1.0</diffuse>
+              <specular>0.2 0.2 0.2 1.0</specular>
+              <emissive>0.0 0.0 0.0 0.0</emissive>
+          </material>
+      </visual>
+  </gazebo>
+  </xacro:macro>
+</robot>

File: ros2_ws/install/yahboom_rosmaster_description/share/yahboom_rosmaster_description/urdf/mech/rosmaster_x3_base.urdf.xacro (robot description, xacro)
@@ -1 +1,56 @@
-/home/amr01/fyp/ros2_ws/src/yahboom_rosmaster/yahboom_rosmaster_description/urdf/mech/rosmaster_x3_base.urdf.xacro
+<?xml version="1.0"?>
+<robot xmlns:xacro="http://www.ros.org/wiki/xacro">
+<xacro:property name="total_width" value="0.19940" />
+<xacro:property name="wheel_width" value="0.0304" />
+<xacro:property name="wheel_radius" value="0.0325" />
+<xacro:property name="total_height" value="0.26225" />
+<xacro:property name="base_length" value="0.300" />
+<xacro:property name="centered_length" value="0.238" />
+<xacro:property name="base_x_offset" value="${(centered_length - base_length) / 2}" />
+<xacro:property name="base_size_x" value="${base_length}" />
+<xacro:property name="base_size_y" value="${total_width - (2 * wheel_width)}" />
+<xacro:property name="base_size_z" value="${total_height - (2 * wheel_radius)}" />
+<xacro:property name="base_mass" value="4.6" />
+<xacro:macro name="rosmaster_x3_base" params="prefix">
+  <link name="${prefix}base_footprint"/>
+  <link name="${prefix}base_link">
+    <visual>
+        <geometry>
+            <mesh filename="file://$(find yahboom_rosmaster_description)/meshes/rosmaster_x3/visual/base_link_X3.STL"/>
+        </geometry>
+        <material name="green">
+          <color rgba="0 0.7 0 1"/>
+        </material>
+        <origin xyz="0 0 0" rpy="0 0 0"/>
+    </visual>
+    <collision>
+        <geometry>
+            <box size="${base_size_x} ${base_size_y} ${base_size_z}"/>
+        </geometry>
+        <origin xyz="${base_x_offset} 0 ${base_size_z/2 + wheel_radius/4}" rpy="0 0 0"/>
+    </collision>
+    <inertial>
+        <origin xyz="${base_x_offset} 0 ${base_size_z/2 + wheel_radius/4}" rpy="0 0 0"/>
+        <mass value="${base_mass}"/>
+        <inertia
+            ixx="${(1/12) * base_mass * ((base_size_y * base_size_y) + (base_size_z * base_size_z))}" ixy="0.0" ixz="0.0"
+            iyy="${(1/12) * base_mass * ((base_size_x * base_size_x) + (base_size_z * base_size_z))}" iyz="0.0"
+            izz="${(1/12) * base_mass * ((base_size_x * base_size_x) + (base_size_y * base_size_y))}"/>
+    </inertial>
+  </link>
+  <gazebo reference="${prefix}base_link">
+    <visual>
+        <material>
+            <ambient>0 0.7 0 1</ambient>
+            <diffuse>0 0.7 0 1</diffuse>
+            <specular>0 0.7 0 1</specular>
+        </material>
+    </visual>
+  </gazebo>
+  <joint name="${prefix}base_joint" type="fixed">
+    <parent link="${prefix}base_footprint"/>
+    <child link="${prefix}base_link"/>
+    <origin xyz="0 0 ${wheel_radius}" rpy="0 0 0"/>
+  </joint>
+</xacro:macro>
+</robot>

File: ros2_ws/install/yahboom_rosmaster_description/share/yahboom_rosmaster_description/urdf/robots/rosmaster_x3.urdf.xacro (robot description, xacro)
@@ -1 +1,65 @@
-/home/amr01/fyp/ros2_ws/src/yahboom_rosmaster/yahboom_rosmaster_description/urdf/robots/rosmaster_x3.urdf.xacro
+<?xml version="1.0"?>
+<robot xmlns:xacro="http://www.ros.org/wiki/xacro" name="rosmaster_x3">
+    <xacro:property name="M_PI" value="3.1415926535897931" />
+    <xacro:arg name="robot_name" default="rosmaster_x3"/>
+    <xacro:arg name="prefix" default=""/>
+    <xacro:arg name="use_gazebo" default="false"/>
+    <xacro:include filename="$(find yahboom_rosmaster_description)/urdf/mech/rosmaster_x3_base.urdf.xacro"/>
+    <xacro:include filename="$(find yahboom_rosmaster_description)/urdf/mech/mecanum_wheel.urdf.xacro"/>
+    <xacro:include filename="$(find yahboom_rosmaster_description)/urdf/sensors/rgbd_camera.urdf.xacro"/>
+    <xacro:include filename="$(find yahboom_rosmaster_description)/urdf/sensors/lidar.urdf.xacro"/>
+    <xacro:include filename="$(find yahboom_rosmaster_description)/urdf/sensors/imu.urdf.xacro"/>
+    <xacro:rosmaster_x3_base prefix="$(arg prefix)"/>
+    <xacro:mecanum_wheel
+      prefix="$(arg prefix)"
+      side="front_left"
+      x_reflect="1"
+      y_reflect="1"/>
+    <xacro:mecanum_wheel
+      prefix="$(arg prefix)"
+      side="front_right"
+      x_reflect="1"
+      y_reflect="-1"/>
+    <xacro:mecanum_wheel
+      prefix="$(arg prefix)"
+      side="back_left"
+      x_reflect="-1"
+      y_reflect="1"/>
+    <xacro:mecanum_wheel
+      prefix="$(arg prefix)"
+      side="back_right"
+      x_reflect="-1"
+      y_reflect="-1"/>
+    <xacro:rgbd_camera
+      prefix="$(arg prefix)"
+      camera_name="cam_1"
+      xyz_offset="0.105 0 0.05"
+      rpy_offset="0 -0.50 0"/>
+    <xacro:lidar_sensor
+      prefix="$(arg prefix)"
+      parent="base_link"
+      frame_id="laser_frame"
+      xyz_offset="0 0 0.0825"
+      rpy_offset="0 0 0"
+      mesh_xyz_offset="0 0 0"
+      mesh_rpy_offset="${-M_PI/2} 0 0"
+      topic_name="scan"/>
+    <xacro:imu_sensor
+      prefix="$(arg prefix)"
+      parent="base_link"
+      frame_id="imu"
+      xyz_offset="0 0 0.006"
+      rpy_offset="0 0 0"
+      update_rate="15.0"
+      topic_name="imu/data"/>
+    <xacro:include filename="$(find yahboom_rosmaster_description)/urdf/control/velocity_control_plugin.urdf.xacro" />
+    <xacro:load_velocity_control_plugin use_gazebo="$(arg use_gazebo)"/>
+    <xacro:include filename="$(find yahboom_rosmaster_description)/urdf/control/gazebo_sim_ros2_control.urdf.xacro" />
+    <xacro:load_gazebo_sim_ros2_control_plugin
+      robot_name="$(arg robot_name)"
+      use_gazebo="$(arg use_gazebo)"/>
+    <xacro:include filename="$(find yahboom_rosmaster_description)/urdf/control/rosmaster_x3_ros2_control.urdf.xacro" />
+    <xacro:yahboom_rosmaster_ros2_control
+      prefix="$(arg prefix)"
+      use_gazebo="$(arg use_gazebo)"/>
+</robot>

File: ros2_ws/install/yahboom_rosmaster_description/share/yahboom_rosmaster_description/urdf/sensors/imu.urdf.xacro (robot description, xacro)
@@ -1 +1,70 @@
-/home/amr01/fyp/ros2_ws/src/yahboom_rosmaster/yahboom_rosmaster_description/urdf/sensors/imu.urdf.xacro
+<?xml version="1.0"?>
+<robot xmlns:xacro="http://www.ros.org/wiki/xacro">
+    <xacro:property name="M_PI" value="3.1415926535897931" />
+    <xacro:macro name="imu_sensor" params="
+        prefix:=''
+        parent:='base_link'
+        frame_id:='imu'
+        xyz_offset:='0 0 0'
+        rpy_offset:='0 0 0'
+        inertial_xyz_offset:='0 0 0'
+        inertial_rpy_offset:='0 0 0'
+        mass:=0.031
+        length:=0.03899
+        width:=0.03785
+        height:=0.01338
+        material_name:='imu_black'
+        material_color:='0.1 0.1 0.1 1'
+        gazebo_material_ambient:='0.1 0.1 0.1 1'
+        gazebo_material_diffuse:='0.1 0.1 0.1 1'
+        gazebo_material_specular:='0.1 0.1 0.1 1'
+        update_rate:='15.0'
+        topic_name:='imu/data'
+        always_on:=true
+        visualize:=false">
+        <xacro:property name="ixx" value="${(mass/12.0) * (height*height + width*width)}" />
+        <xacro:property name="iyy" value="${(mass/12.0) * (length*length + height*height)}" />
+        <xacro:property name="izz" value="${(mass/12.0) * (length*length + width*width)}" />
+        <link name="${prefix}${frame_id}_link">
+            <visual>
+                <origin xyz="0 0 0" rpy="0 0 0"/>
+                <geometry>
+                    <box size="${length} ${width} ${height}"/>
+                </geometry>
+                <material name="${material_name}">
+                    <color rgba="${material_color}"/>
+                </material>
+            </visual>
+            <inertial>
+                <mass value="${mass}" />
+                <origin xyz="${inertial_xyz_offset}" rpy="${inertial_rpy_offset}"/>
+                <inertia
+                    ixx="${ixx}"
+                    ixy="0.0"
+                    ixz="0.0"
+                    iyy="${iyy}"
+                    iyz="0.0"
+                    izz="${izz}" />
+            </inertial>
+        </link>
+        <joint name="${prefix}${frame_id}_joint" type="fixed">
+            <parent link="${prefix}${parent}"/>
+            <child link="${prefix}${frame_id}_link" />
+            <origin xyz="${xyz_offset}" rpy="${rpy_offset}"/>
+        </joint>
+        <gazebo reference="${prefix}${frame_id}_link">
+            <material>
+                <ambient>${gazebo_material_ambient}</ambient>
+                <diffuse>${gazebo_material_diffuse}</diffuse>
+                <specular>${gazebo_material_specular}</specular>
+            </material>
+            <sensor name="${prefix}imu_sensor" type="imu">
+                <topic>${topic_name}</topic>
+                <update_rate>${update_rate}</update_rate>
+                <always_on>${always_on}</always_on>
+                <visualize>${visualize}</visualize>
+                <gz_frame_id>${prefix}${frame_id}_link</gz_frame_id>
+            </sensor>
+        </gazebo>
+    </xacro:macro>
+</robot>

File: ros2_ws/install/yahboom_rosmaster_description/share/yahboom_rosmaster_description/urdf/sensors/lidar.urdf.xacro (robot description, xacro)
@@ -1 +1,111 @@
-/home/amr01/fyp/ros2_ws/src/yahboom_rosmaster/yahboom_rosmaster_description/urdf/sensors/lidar.urdf.xacro
+<?xml version="1.0"?>
+<robot xmlns:xacro="http://www.ros.org/wiki/xacro">
+  <xacro:property name="M_PI" value="3.1415926535897931" />
+  <xacro:macro name="lidar_sensor" params="
+    prefix:=''
+    parent:='base_link'
+    frame_id:='laser_frame'
+    mesh_file:='file://$(find yahboom_rosmaster_description)/meshes/rplidar/rplidar_s2.stl'
+    xyz_offset:='0 0 0.0825'
+    rpy_offset:='0 0 0'
+    mesh_xyz_offset:='0 0 0'
+    mesh_rpy_offset:='${-M_PI/2} 0 0'
+    mesh_scale:='0.001 0.001 0.001'
+    collision_xyz_offset:='0 0 0'
+    collision_rpy_offset:='0 0 0'
+    inertial_xyz_offset:='0 0 0'
+    inertial_rpy_offset:='0 0 0'
+    lidar_width:=0.077
+    lidar_height:=0.0398
+    mass:=0.185
+    material_name:='rplidar_black'
+    material_color:='0.1 0.1 0.1 1'
+    gazebo_material_ambient:='0.1 0.1 0.1 1'
+    gazebo_material_diffuse:='0.1 0.1 0.1 1'
+    gazebo_material_specular:='0.1 0.1 0.1 1'
+    update_rate:=10
+    ray_count:=720
+    min_angle:='-3.14159'
+    max_angle:='3.14159'
+    min_range:='0.20'
+    max_range:='30.0'
+    range_resolution:='0.013'
+    topic_name:='scan'
+    always_on:=true
+    visualize:=false
+    enable_collision:=false">
+    <xacro:property name="radius" value="${lidar_width/2}" />
+    <xacro:property name="ixx_iyy" value="${(mass/12) * (3 * radius * radius + lidar_height * lidar_height)}" />
+    <xacro:property name="izz" value="${(mass/2) * (radius * radius)}" />
+    <link name="${prefix}${frame_id}">
+      <visual>
+        <origin xyz="${mesh_xyz_offset}" rpy="${mesh_rpy_offset}"/>
+        <geometry>
+          <mesh filename="${mesh_file}" scale="${mesh_scale}"/>
+        </geometry>
+        <material name="${material_name}">
+          <color rgba="${material_color}"/>
+        </material>
+      </visual>
+      <xacro:if value="${enable_collision}">
+        <collision>
+          <origin xyz="${collision_xyz_offset}" rpy="${collision_rpy_offset}"/>
+          <geometry>
+            <cylinder radius="${lidar_width/2}" length="${lidar_height}"/>
+          </geometry>
+        </collision>
+      </xacro:if>
+      <inertial>
+        <mass value="${mass}" />
+        <origin xyz="${inertial_xyz_offset}" rpy="${inertial_rpy_offset}"/>
+        <inertia
+          ixx="${ixx_iyy}"
+          ixy="0.0"
+          ixz="0.0"
+          iyy="${ixx_iyy}"
+          iyz="0.0"
+          izz="${izz}" />
+      </inertial>
+    </link>
+    <joint name="${prefix}${frame_id}_joint" type="fixed">
+      <parent link="${prefix}${parent}"/>
+      <child link="${prefix}${frame_id}" />
+      <origin xyz="${xyz_offset}" rpy="${rpy_offset}"/>
+    </joint>
+    <gazebo reference="${prefix}${frame_id}">
+      <material>
+        <ambient>${gazebo_material_ambient}</ambient>
+        <diffuse>${gazebo_material_diffuse}</diffuse>
+        <specular>${gazebo_material_specular}</specular>
+      </material>
+      <sensor name="${prefix}lidar_sensor" type="gpu_lidar">
+        <topic>${topic_name}</topic>
+        <update_rate>${update_rate}</update_rate>
+        <always_on>${always_on}</always_on>
+        <visualize>${visualize}</visualize>
+        <ray>
+          <scan>
+            <horizontal>
+              <samples>${ray_count}</samples>
+              <resolution>1</resolution>
+              <min_angle>${min_angle}</min_angle>
+              <max_angle>${max_angle}</max_angle>
+            </horizontal>
+            <vertical>
+              <samples>1</samples>
+              <resolution>1</resolution>
+              <min_angle>0</min_angle>
+              <max_angle>0</max_angle>
+            </vertical>
+          </scan>
+          <range>
+            <min>${min_range}</min>
+            <max>${max_range}</max>
+            <resolution>${range_resolution}</resolution>
+          </range>
+        </ray>
+        <gz_frame_id>${prefix}${frame_id}</gz_frame_id>
+      </sensor>
+    </gazebo>
+  </xacro:macro>
+</robot>
